File: hw/gb_rp2040_cart.kicad_sch (KiCad schematic)
At the start: 14 parts, among them J1 GameBoy_Cartridge, U1 SN74LVC8T245PW, U2 SN74LVC8T245PW, U3 TXU0104, U4 SN74LVC8T245PW

Commit message: hw: add more information to BOM
Signed-off-by: Mahyar Koshkouei <mk@deltabeard.com>
Parts:
- C1, C2, C3, C4, C5, C6, C7, C8: MFr (none) -> CL05B104KO5NNNC; Manufacturer (none) -> Samsung Electro-Mechanics; Notes (none) -> Alternative manufacturer is acceptable
- J1, TP1: Notes (none) -> Only footprint, no component.
- U1, U2, U4: MFr (none) -> SN74LVC8T245PWR; Manufacturer (none) -> Texas Instruments
- U3: Notes (none) -> Do not populate.
Changed lines of the file:
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@@
+      (effects (font (size 1.27 1.27)) hide)
+    )
+    (property "Notes" "Only footprint, no component." (id 4) (at 44.45 56.515 0)
       (effects (font (size 1.27 1.27)) hide)
     )
@@
       (effects (font (size 1.27 1.27)) hide)
     )
+    (property "MFr" "CL05B104KO5NNNC" (id 5) (at 86.36 107.95 0)
+      (effects (font (size 1.27 1.27)) hide)
+    )
+    (property "Manufacturer" "Samsung Electro-Mechanics " (id 6) (at 86.36 107.95 0)
+      (effects (font (size 1.27 1.27)) hide)
+    )
+    (property "Notes" "Alternative manufacturer is acceptable" (id 7) (at 86.36 107.95 0)
+      (effects (font (size 1.27 1.27)) hide)
+    )
+    (property "Description" " X7R 100nF ±10% 16V 0402 Multilayer Ceramic Capacitors MLCC - SMD/SMT ROHS " (id 8) (at 86.36 107.95 0)
+      (effects (font (size 1.27 1.27)) hide)
+    )
     (pin "1")
     (pin "2")
@@
       (effects (font (size 1.27 1.27)) hide)
     )
+    (property "MFr" "CL05B104KO5NNNC" (id 5) (at 86.995 40.005 0)
+      (effects (font (size 1.27 1.27)) hide)
+    )
+    (property "Manufacturer" "Samsung Electro-Mechanics " (id 6) (at 86.995 40.005 0)
+      (effects (font (size 1.27 1.27)) hide)
+    )
+    (property "Notes" "Alternative manufacturer is acceptable" (id 7) (at 86.995 40.005 0)
+      (effects (font (size 1.27 1.27)) hide)
+    )
+    (property "Description" " X7R 100nF ±10% 16V 0402 Multilayer Ceramic Capacitors MLCC - SMD/SMT ROHS " (id 8) (at 86.995 40.005 0)
+      (effects (font (size 1.27 1.27)) hide)
+    )
     (pin "1")
     (pin "2")
@@
       (effects (font (size 1.27 1.27)) hide)
     )
+    (property "MFr" "CL05B104KO5NNNC" (id 5) (at 105.41 107.95 0)
+      (effects (font (size 1.27 1.27)) hide)
+    )
+    (property "Manufacturer" "Samsung Electro-Mechanics " (id 6) (at 105.41 107.95 0)
+      (effects (font (size 1.27 1.27)) hide)
+    )
+    (property "Notes" "Alternative manufacturer is acceptable" (id 7) (at 105.41 107.95 0)
+      (effects (font (size 1.27 1.27)) hide)
+    )
+    (property "Description" " X7R 100nF ±10% 16V 0402 Multilayer Ceramic Capacitors MLCC - SMD/SMT ROHS " (id 8) (at 105.41 107.95 0)
+      (effects (font (size 1.27 1.27)) hide)
+    )
     (pin "1")
     (pin "2")
@@
       (effects (font (size 1.27 1.27)) hide)
     )
+    (property "MFr" "CL05B104KO5NNNC" (id 5) (at 106.045 40.005 0)
+      (effects (font (size 1.27 1.27)) hide)
+    )
+    (property "Manufacturer" "Samsung Electro-Mechanics " (id 6) (at 106.045 40.005 0)
+      (effects (font (size 1.27 1.27)) hide)
+    )
+    (property "Notes" "Alternative manufacturer is acceptable" (id 7) (at 106.045 40.005 0)
+      (effects (font (size 1.27 1.27)) hide)
+    )
+    (property "Description" " X7R 100nF ±10% 16V 0402 Multilayer Ceramic Capacitors MLCC - SMD/SMT ROHS " (id 8) (at 106.045 40.005 0)
+      (effects (font (size 1.27 1.27)) hide)
+    )
     (pin "1")
     (pin "2")
@@
       (effects (font (size 1.27 1.27)) hide)
     )
+    (property "MFr" "CL05B104KO5NNNC" (id 5) (at 170.815 36.195 0)
+      (effects (font (size 1.27 1.27)) hide)
+    )
+    (property "Manufacturer" "Samsung Electro-Mechanics " (id 6) (at 170.815 36.195 0)
+      (effects (font (size 1.27 1.27)) hide)
+    )
+    (property "Notes" "Alternative manufacturer is acceptable" (id 7) (at 170.815 36.195 0)
+      (effects (font (size 1.27 1.27)) hide)
+    )
+    (property "Description" " X7R 100nF ±10% 16V 0402 Multilayer Ceramic Capacitors MLCC - SMD/SMT ROHS " (id 8) (at 170.815 36.195 0)
+      (effects (font (size 1.27 1.27)) hide)
+    )
     (pin "1")
     (pin "2")
@@
       (effects (font (size 1.27 1.27)) hide)
     )
+    (property "MFr" "CL05B104KO5NNNC" (id 5) (at 171.45 114.935 0)
+      (effects (font (size 1.27 1.27)) hide)
+    )
+    (property "Manufacturer" "Samsung Electro-Mechanics " (id 6) (at 171.45 114.935 0)
+      (effects (font (size 1.27 1.27)) hide)
+    )
+    (property "Notes" "Alternative manufacturer is acceptable" (id 7) (at 171.45 114.935 0)
+      (effects (font (size 1.27 1.27)) hide)
+    )
+    (property "Description" " X7R 100nF ±10% 16V 0402 Multilayer Ceramic Capacitors MLCC - SMD/SMT ROHS " (id 8) (at 171.45 114.935 0)
+      (effects (font (size 1.27 1.27)) hide)
+    )
     (pin "1")
     (pin "2")
@@
       (effects (font (size 1.27 1.27)) hide)
     )
+    (property "MFr" "CL05B104KO5NNNC" (id 5) (at 189.865 36.195 0)
+      (effects (font (size 1.27 1.27)) hide)
+    )
+    (property "Manufacturer" "Samsung Electro-Mechanics " (id 6) (at 189.865 36.195 0)
+      (effects (font (size 1.27 1.27)) hide)
+    )
+    (property "Notes" "Alternative manufacturer is acceptable" (id 7) (at 189.865 36.195 0)
+      (effects (font (size 1.27 1.27)) hide)
+    )
+    (property "Description" " X7R 100nF ±10% 16V 0402 Multilayer Ceramic Capacitors MLCC - SMD/SMT ROHS " (id 8) (at 189.865 36.195 0)
+      (effects (font (size 1.27 1.27)) hide)
+    )
     (pin "1")
     (pin "2")
@@
     )
     (property "LCSC" "C1525" (id 4) (at 190.5 114.935 0)
+      (effects (font (size 1.27 1.27)) hide)
+    )
+    (property "MFr" "CL05B104KO5NNNC" (id 5) (at 190.5 114.935 0)
+      (effects (font (size 1.27 1.27)) hide)
+    )
+    (property "Manufacturer" "Samsung Electro-Mechanics " (id 6) (at 190.5 114.935 0)
+      (effects (font (size 1.27 1.27)) hide)
+    )
+    (property "Notes" "Alternative manufacturer is acceptable" (id 7) (at 190.5 114.935 0)
+      (effects (font (size 1.27 1.27)) hide)
+    )
+    (property "Description" " X7R 100nF ±10% 16V 0402 Multilayer Ceramic Capacitors MLCC - SMD/SMT ROHS " (id 8) (at 190.5 114.935 0)
       (effects (font (size 1.27 1.27)) hide)
     )
@@
     )
     (property "Datasheet" "https://www.ti.com/lit/ds/symlink/txu0104.pdf" (id 3) (at 180.34 159.385 0)
+      (effects (font (size 1.27 1.27)) hide)
+    )
+    (property "Notes" "Do not populate." (id 4) (at 180.34 131.445 0)
       (effects (font (size 1.27 1.27)) hide)
     )
@@
     (property "Datasheet" "" (id 3) (at 26.67 97.155 0)
       (effects (font (size 1.27 1.27)) (justify left) hide)
+    )
+    (property "Notes" "Only footprint, no component." (id 4) (at 26.67 97.155 0)
+      (effects (font (size 1.27 1.27)) hide)
     )
     (pin "1")
@@
       (effects (font (size 1.27 1.27)) hide)
     )
+    (property "Description" " TSSOP-24 Translators / Level Shifters ROHS " (id 5) (at 95.25 132.08 0)
+      (effects (font (size 1.27 1.27)) hide)
+    )
+    (property "MFr" "SN74LVC8T245PWR" (id 6) (at 95.25 132.08 0)
+      (effects (font (size 1.27 1.27)) hide)
+    )
+    (property "Manufacturer" " Texas Instruments " (id 7) (at 95.25 132.08 0)
+      (effects (font (size 1.27 1.27)) hide)
+    )
     (pin "1")
     (pin "10")
@@
       (effects (font (size 1.27 1.27)) hide)
     )
+    (property "Description" " TSSOP-24 Translators / Level Shifters ROHS " (id 5) (at 95.885 64.135 0)
+      (effects (font (size 1.27 1.27)) hide)
+    )
+    (property "MFr" "SN74LVC8T245PWR" (id 6) (at 95.885 64.135 0)
+      (effects (font (size 1.27 1.27)) hide)
+    )
+    (property "Manufacturer" " Texas Instruments " (id 7) (at 95.885 64.135 0)
+      (effects (font (size 1.27 1.27)) hide)
+    )
     (pin "1")
     (pin "10")
@@
       (effects (font (size 1.27 1.27)) hide)
     )
+    (property "Description" " TSSOP-24 Translators / Level Shifters ROHS " (id 5) (at 180.975 60.325 0)
+      (effects (font (size 1.27 1.27)) hide)
+    )
+    (property "MFr" "SN74LVC8T245PWR" (id 6) (at 180.975 60.325 0)
+      (effects (font (size 1.27 1.27)) hide)
+    )
+    (property "Manufacturer" " Texas Instruments " (id 7) (at 180.975 60.325 0)
+      (effects (font (size 1.27 1.27)) hide)
+    )
