File: hw/gb_rp2040_cart.kicad_sch (KiCad schematic)
At the start: 14 parts, among them J1 GameBoy_Cartridge, U1 SN74LVC8T245PW, U2 SN74LVC8T245PW, U3 TXU0104, U4 SN74LVC8T245PW

Commit message: all: Add open source license
Signed-off-by: Mahyar Koshkouei <mk@deltabeard.com>
Other:
- company: Mahyar Koshkouei -> Copyright (c) 2021 Mahyar Koshkouei
- title: RP2040 Game Boy Cart -> DBGC: RP2040 Game Boy Cart
Changed lines of the file:
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@@
   (paper "A4")
   (title_block
-    (title "RP2040 Game Boy Cart")
+    (title "DBGC: RP2040 Game Boy Cart")
     (date "2021-09-29")
     (rev "0.3a")
-    (company "Mahyar Koshkouei")
-    (comment 1 "All Rights Reserved")
+    (company "Copyright (c) 2021 Mahyar Koshkouei")
+    (comment 1 "CC BY-SA 4.0")
     (comment 2 "Compatible with DMG, MGB, & CGB. Collectively referred to as \"GB\" here.")
   )
