File: hw/peripherals.kicad_sch (KiCad schematic)
At the start: 22 parts, among them Q2 N-Channel, SW1 SW_DPST, U10 MB85RC256VPNF-G-JNERE1, U11 DS3231M, U9 PCA9536D

Commit message: hw: add more information to BOM
Signed-off-by: Mahyar Koshkouei <mk@deltabeard.com>
Parts:
- BT1: MFr (none) -> MY-2032-11; Manufacturer (none) -> MYOUNG
- C23, C24, C25: MFr (none) -> CL05B104KO5NNNC; Manufacturer (none) -> Samsung Electro-Mechanics; Notes (none) -> Alternative manufacturer is acceptable
- D2: MFr (none) -> KT-0603R; Notes (none) -> Alternative manufacturer is acceptable
- Q2: Manufacturer (none) -> Changjiang Electronics Tech (CJ); Notes (none) -> Alternative manufacturer is acceptable
- R10, R9: MFr (none) -> 0402WGF4701TCE; Manufacturer (none) -> UNI-ROYAL(Uniroyal Elec); Notes (none) -> Alternative manufacturer is acceptable
- R11, R13: MFr (none) -> 0603WAF3300T5E; Manufacturer (none) -> UNI-ROYAL(Uniroyal Elec); Notes (none) -> Alternative manufacturer is acceptable
- R12, R14: MFr (none) -> 0603WAF1003T5E; Manufacturer (none) -> UNI-ROYAL(Uniroyal Elec); Notes (none) -> Alternative manufacturer is acceptable
- SW1: Manufacturer (none) -> Korean Hroparts Elec
- TP40, TP41, TP42, TP43, TP44, TP45: Notes (none) -> Only footprint, no component.
- U10: MFr (none) -> MB85RC256VPNF-G-JNERE1; Manufacturer (none) -> FUJITSU
- U11: MFr (none) -> DS3231M+TRL; Manufacturer (none) -> Maxim Integrated
- U9: MFr (none) -> PCA9536D; Manufacturer (none) -> NXP Semicon; Notes (none) -> Do not populate.

Commit message: hw: fix USB
Additionally reduced the size of the battery holder.

Signed-off-by: Mahyar Koshkouei <mk@deltabeard.com>
Parts:
- BT1: footprint Battery:BatteryHolder_MPD_BC2003_1x2032 -> Battery:BatteryHolder_Keystone_3000_1x12mm; LCSC C964835 -> C964818; MFr MY-2032-11 -> MY-1220-03
Changed lines of the file:
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@@
       (effects (font (size 1.27 1.27)) (justify left))
     )
-    (property "Footprint" "Battery:BatteryHolder_MPD_BC2003_1x2032" (id 2) (at 84.455 53.721 90)
+    (property "Footprint" "Battery:BatteryHolder_Keystone_3000_1x12mm" (id 2) (at 84.455 53.721 90)
       (effects (font (size 1.27 1.27)) hide)
     )
@@
       (effects (font (size 1.27 1.27)) hide)
     )
-    (property "LCSC" "C964835" (id 4) (at 84.455 55.245 0)
+    (property "LCSC" "C964818" (id 4) (at 84.455 55.245 0)
       (effects (font (size 1.27 1.27)) hide)
     )
-    (property "MFr" "MY-2032-11" (id 5) (at 84.455 55.245 0)
+    (property "MFr" "MY-1220-03" (id 5) (at 84.455 55.245 0)
       (effects (font (size 1.27 1.27)) hide)
     )
@@
       (effects (font (size 1.27 1.27)) hide)
     )
-    (property "Description" "CR2032 Battery holder" (id 8) (at 84.455 55.245 0)
+    (property "Description" "CR1220 Battery holder" (id 8) (at 84.455 55.245 0)
       (effects (font (size 1.27 1.27)) hide)
     )

Commit message: hw: add BOOTSEL button and routing changes
Signed-off-by: Mahyar Koshkouei <mk@deltabeard.com>
Parts:
- U9: Manufacturer NXP Semicon -> NXP Semicon; Notes Do not populate. -> Do not populate. Do not use Texas Instruments version due t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
Changed lines of the file:
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@@
   (title_block
     (title "RP2040 Game Boy Cart")
-    (date "2021-08-31")
-    (rev "0.2a")
+    (date "2021-09-29")
+    (rev "0.3a")
     (company "Mahyar Koshkouei")
     (comment 1 "All Rights Reserved")
@@
       (effects (font (size 1.27 1.27)) hide)
     )
-    (property "Description" " 4 POR I?C, SMBus 400kHz SOIC-8 I/O Expanders ROHS " (id 5) (at 100.33 115.57 0)
+    (property "Description" "4 POR I?C, SMBus 400kHz SOIC-8 I/O Expanders ROHS " (id 5) (at 100.33 115.57 0)
       (effects (font (size 1.27 1.27)) hide)
     )
@@
       (effects (font (size 1.27 1.27)) hide)
     )
-    (property "Manufacturer" " NXP Semicon " (id 7) (at 100.33 115.57 0)
-      (effects (font (size 1.27 1.27)) hide)
-    )
-    (property "Notes" "Do not populate." (id 8) (at 100.33 115.57 0)
-      (effects (font (size 1.27 1.27)) hide)
-    )
+    (property "Manufacturer" "NXP Semicon " (id 7) (at 100.33 115.57 0)
+      (effects (font (size 1.27 1.27)) hide)
+    )
+    (property "Notes" "Do not populate. Do not use Texas Instruments version due to VPOR errata." (id 8) (at 100.33 115.57 0)
+      (effects (font (size 1.27 1.27)) hide)
+    )
