File: hw/power.kicad_sch (KiCad schematic)
At the start: 6 parts, among them Q1 SI2301CDS-T1-GE3, U7 XC6206P332MR

Commit message: hw: WIP
Signed-off-by: Mahyar Koshkouei <mk@deltabeard.com>
Parts:
- C23, C24: footprint Capacitor_SMD:C_0603_1608Metric -> Capacitor_SMD:C_0402_1005Metric; LCSC C15849 -> C52923; MFr CL10A105KB8NNNC -> CL05A105KA5NQNC; Manufacturer Samsung Electro-Mechanics -> Samsung Electro-Mechanics
- R10: renamed from R11; Manufacturer UNI-ROYAL(Uniroyal Elec) -> UNI-ROYAL(Uniroyal Elec)
Changed lines of the file:
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@@
   (symbol (lib_id "power:VBUS") (at 113.665 77.47 90) (unit 1)
     (in_bom yes) (on_board yes)
-    (property "Reference" "#PWR064" (id 0) (at 117.475 77.47 0)
+    (property "Reference" "#PWR062" (id 0) (at 117.475 77.47 0)
       (effects (font (size 1.27 1.27)) hide)
     )
@@
   (symbol (lib_id "power:+5V") (at 150.495 73.66 0) (unit 1)
     (in_bom yes) (on_board yes) (fields_autoplaced)
-    (property "Reference" "#PWR066" (id 0) (at 150.495 77.47 0)
+    (property "Reference" "#PWR064" (id 0) (at 150.495 77.47 0)
       (effects (font (size 1.27 1.27)) hide)
     )
@@
   (symbol (lib_id "power:+3V3") (at 188.595 77.47 270) (unit 1)
     (in_bom yes) (on_board yes) (fields_autoplaced)
-    (property "Reference" "#PWR068" (id 0) (at 184.785 77.47 0)
+    (property "Reference" "#PWR066" (id 0) (at 184.785 77.47 0)
       (effects (font (size 1.27 1.27)) hide)
     )
@@
   (symbol (lib_id "power:GND") (at 116.84 106.68 0) (unit 1)
     (in_bom yes) (on_board yes) (fields_autoplaced)
-    (property "Reference" "#PWR065" (id 0) (at 116.84 113.03 0)
+    (property "Reference" "#PWR063" (id 0) (at 116.84 113.03 0)
       (effects (font (size 1.27 1.27)) hide)
     )
@@
   (symbol (lib_id "power:GND") (at 170.18 90.17 0) (unit 1)
     (in_bom yes) (on_board yes) (fields_autoplaced)
-    (property "Reference" "#PWR067" (id 0) (at 170.18 96.52 0)
+    (property "Reference" "#PWR065" (id 0) (at 170.18 96.52 0)
       (effects (font (size 1.27 1.27)) hide)
     )
@@
   (symbol (lib_id "Device:R_Small") (at 116.84 102.87 0) (unit 1)
     (in_bom yes) (on_board yes)
-    (property "Reference" "R11" (id 0) (at 118.11 102.2349 0)
+    (property "Reference" "R10" (id 0) (at 118.11 102.2349 0)
       (effects (font (size 1.27 1.27)) (justify left))
     )
@@
       (effects (font (size 1.27 1.27)) hide)
     )
-    (property "Manufacturer" " UNI-ROYAL(Uniroyal Elec) " (id 8) (at 116.84 102.87 0)
+    (property "Manufacturer" "UNI-ROYAL(Uniroyal Elec) " (id 8) (at 116.84 102.87 0)
       (effects (font (size 1.27 1.27)) hide)
     )
@@
       (effects (font (size 1.27 1.27)) (justify left))
     )
-    (property "Footprint" "Capacitor_SMD:C_0603_1608Metric" (id 2) (at 154.94 81.28 0)
+    (property "Footprint" "Capacitor_SMD:C_0402_1005Metric" (id 2) (at 154.94 81.28 0)
       (effects (font (size 1.27 1.27)) hide)
     )
@@
       (effects (font (size 1.27 1.27)) hide)
     )
-    (property "LCSC" "C15849" (id 4) (at 154.94 81.28 0)
+    (property "LCSC" "C52923" (id 4) (at 154.94 81.28 0)
       (effects (font (size 1.27 1.27)) hide)
     )
-    (property "Description" " X5R ±10% 50V 1uF 0603 Multilayer Ceramic Capacitors MLCC - SMD/SMT ROHS " (id 5) (at 154.94 81.28 0)
+    (property "Description" "X5R 25V ±10% 1uF 0402 Multilayer Ceramic Capacitors MLCC - SMD/SMT ROHS" (id 5) (at 154.94 81.28 0)
       (effects (font (size 1.27 1.27)) hide)
     )
-    (property "MFr" "CL10A105KB8NNNC" (id 6) (at 154.94 81.28 0)
+    (property "MFr" "CL05A105KA5NQNC" (id 6) (at 154.94 81.28 0)
       (effects (font (size 1.27 1.27)) hide)
     )
-    (property "Manufacturer" " Samsung Electro-Mechanics " (id 7) (at 154.94 81.28 0)
+    (property "Manufacturer" "Samsung Electro-Mechanics " (id 7) (at 154.94 81.28 0)
       (effects (font (size 1.27 1.27)) hide)
     )
@@
       (effects (font (size 1.27 1.27)) (justify left))
     )
-    (property "Footprint" "Capacitor_SMD:C_0603_1608Metric" (id 2) (at 181.61 81.28 0)
+    (property "Footprint" "Capacitor_SMD:C_0402_1005Metric" (id 2) (at 181.61 81.28 0)
       (effects (font (size 1.27 1.27)) hide)
     )
@@
       (effects (font (size 1.27 1.27)) hide)
     )
-    (property "LCSC" "C15849" (id 4) (at 181.61 81.28 0)
+    (property "LCSC" "C52923" (id 4) (at 181.61 81.28 0)
       (effects (font (size 1.27 1.27)) hide)
     )
-    (property "Description" " X5R ±10% 50V 1uF 0603 Multilayer Ceramic Capacitors MLCC - SMD/SMT ROHS " (id 5) (at 181.61 81.28 0)
+    (property "Description" "X5R 25V ±10% 1uF 0402 Multilayer Ceramic Capacitors MLCC - SMD/SMT ROHS" (id 5) (at 181.61 81.28 0)
       (effects (font (size 1.27 1.27)) hide)
     )
-    (property "MFr" "CL10A105KB8NNNC" (id 6) (at 181.61 81.28 0)
+    (property "MFr" "CL05A105KA5NQNC" (id 6) (at 181.61 81.28 0)
       (effects (font (size 1.27 1.27)) hide)
     )
-    (property "Manufacturer" " Samsung Electro-Mechanics " (id 7) (at 181.61 81.28 0)
+    (property "Manufacturer" "Samsung Electro-Mechanics " (id 7) (at 181.61 81.28 0)
       (effects (font (size 1.27 1.27)) hide)
     )
